Commit message: modify soma mse pkg

File: soma_mse/xacro/movebase_macro.xacro (robot description, xacro)
@@ -38,5 +38,5 @@
 			<inertial>
 				<origin xyz="0.0 0.0 0.0" rpy="0.0 0.0 0.0" />
-				<mass value="0.1" />
+				<mass value="0.5" />
 				<inertia ixx="0.0001" ixy="0.0" ixz="0.0" iyy="0.0001" iyz="0.0" izz="0.0001" />
 			</inertial>

Commit message: update simulator
robot description and local planner parameters

File: soma_mse/xacro/movebase_macro.xacro (robot description, xacro)
@@ -43,5 +43,5 @@
 			<visual>
 				<geometry>
-					<cylinder radius="0.05" length="0.02" />
+					<cylinder radius="0.2" length="0.1" />
 				</geometry>
 				<material name="red" />
@@ -49,5 +49,5 @@
 			<collision>
 				<geometry>
-					<cylinder radius="0.05" length="0.02" />
+					<cylinder radius="0.2" length="0.1" />
 				</geometry>
 			</collision>
@@ -69,5 +69,5 @@
 			<parent link="${parent}" />
 			<child link="body_link" />
-			<origin xyz="-0.07 0 0.07" rpy="0.0 0.0 0.0" />
+			<origin xyz="0 0 0.4" rpy="0.0 0.0 0.0" />
 		</joint>
 		<link name="body_link">
@@ -80,5 +80,5 @@
 				<origin xyz="0.0 0.0 0.0" rpy="0.0 0.0 0.0" />
 				<geometry>
-					<box size="0.24 0.18 0.06" />
+					<box size="0.6 0.40 0.6" />
 				</geometry>
 				<material name="gray" />
@@ -87,5 +87,5 @@
 				<origin xyz="0.0 0.0 0.0" rpy="0.0 0.0 0.0" />
 				<geometry>
-					<box size="0.24 0.178 0.06" />
+					<box size="0.6 0.40 0.6" />
 				</geometry>
 			</collision>
@@ -101,5 +101,5 @@
 			<parent link="${parent}" />
 			<child link="ball_link" />
-			<origin xyz="-0.14 0 0.04" rpy="0.0 0.0 0.0" />
+			<origin xyz="-0.14 0 0.1" rpy="0.0 0.0 0.0" />
 		</joint>
 		<link name="ball_link">
@@ -107,5 +107,5 @@
 				<origin xyz="0.0 0.0 0.0" rpy="0.0 0.0 0.0" />
 				<geometry>
-					<sphere radius="0.04" />
+					<sphere radius="0.1" />
 				</geometry>
 				<material name="gray" />
@@ -114,5 +114,5 @@
 				<origin xyz="0.0 0.0 0.0" rpy="0.0 0.0 0.0" />
 				<geometry>
-					<sphere radius="0.04" />
+					<sphere radius="0.1" />
 				</geometry>
 				<material name="gray" />

File: soma_mse/xacro/movebase_vlp16.xacro (robot description, xacro)
@@ -7,10 +7,10 @@
 	<!--  -->
 	<body_macro parent="base_link" />
-	<wheel_macro prefix="left_wheel" parent="base_link" xyz="0 0.1 0.05" />
-	<wheel_macro prefix="right_wheel" parent="base_link" xyz="0 -0.1 0.05" />
+	<wheel_macro prefix="left_wheel" parent="base_link" xyz="0.2 0.3 0.2" />
+	<wheel_macro prefix="right_wheel" parent="base_link" xyz="0.2 -0.3 0.2" />
 	<!--  -->
 	<!--  -->
 	<VLP-16>
-		<origin xyz="0.0 0.0 0.10" rpy="0.0 0.0 0.0" />
+		<origin parent="base_link" xyz="0.25 0.0 0.7" rpy="0.0 0.0 0.0" />
 	</VLP-16>
 	<!--  -->
